Commit message: slight syntax change

File: src/arm/arm_description/urdf/my_arm.xacro (robot description, xacro)
@@ -10,4 +10,19 @@
 <!-- base_link -->
 <link name="base_link">
+    <visual>
+      <geometry>
+            <box size = "0.1 0.1 0.1"/>
+        </geometry>
+        <material name="blue">
+            <color rgba="0 0 .8 1"/>
+        </material>
+        <origin xyz="0 0 0"/>
+    </visual>
+    <collision>
+      <geometry>
+            <box size = "0.1 0.1 0.1"/>
+        </geometry>
+        <origin xyz="0 0 0"/>
+    </collision>
     <inertial>
       <mass value="2e-06"/>
@@ -162,52 +177,52 @@
 <!-- Transmission -->
 <transmission name="tran1">
-<type>transmission_interface/SimpleTransmission</type>
-<joint name="base">
-  <hardwareInterface>EffortJointInterface</hardwareInterface>
-</joint>
-<actuator name="motor1">
-  <hardwareInterface>EffortJointInterface</hardwareInterface>
-  <mechanicalReduction>1</mechanicalReduction>
-</actuator>
+  <type>transmission_interface/SimpleTransmission</type>
+  <joint name="base">
+    <hardwareInterface>EffortJointInterface</hardwareInterface>
+  </joint>
+  <actuator name="motor1">
+    <hardwareInterface>EffortJointInterface</hardwareInterface>
+    <mechanicalReduction>1</mechanicalReduction>
+  </actuator>
 </transmission>
 <transmission name="tran2">
-<type>transmission_interface/SimpleTransmission</type>
-<joint name="elbow">
-  <hardwareInterface>EffortJointInterface</hardwareInterface>
-</joint>
-<actuator name="motor2">
-  <hardwareInterface>EffortJointInterface</hardwareInterface>
-  <mechanicalReduction>1</mechanicalReduction>
-</actuator>
+  <type>transmission_interface/SimpleTransmission</type>
+  <joint name="elbow">
+    <hardwareInterface>EffortJointInterface</hardwareInterface>
+  </joint>
+  <actuator name="motor2">
+    <hardwareInterface>EffortJointInterface</hardwareInterface>
+    <mechanicalReduction>1</mechanicalReduction>
+  </actuator>
 </transmission>
 <transmission name="tran3">
-<type>transmission_interface/SimpleTransmission</type>
-<joint name="wist">
-  <hardwareInterface>EffortJointInterface</hardwareInterface>
-</joint>
-<actuator name="motor3">
-  <hardwareInterface>EffortJointInterface</hardwareInterface>
-  <mechanicalReduction>1</mechanicalReduction>
-</actuator>
+  <type>transmission_interface/SimpleTransmission</type>
+  <joint name="wist">
+    <hardwareInterface>EffortJointInterface</hardwareInterface>
+  </joint>
+  <actuator name="motor3">
+    <hardwareInterface>EffortJointInterface</hardwareInterface>
+    <mechanicalReduction>1</mechanicalReduction>
+  </actuator>
 </transmission>
 <transmission name="tran4">
-<type>transmission_interface/SimpleTransmission</type>
-<joint name="hand_to_right_finger">
-  <hardwareInterface>EffortJointInterface</hardwareInterface>
-</joint>
-<actuator name="motor4">
-  <hardwareInterface>EffortJointInterface</hardwareInterface>
-  <mechanicalReduction>1</mechanicalReduction>
-</actuator>
+  <type>transmission_interface/SimpleTransmission</type>
+  <joint name="hand_to_right_finger">
+    <hardwareInterface>EffortJointInterface</hardwareInterface>
+  </joint>
+  <actuator name="motor4">
+    <hardwareInterface>EffortJointInterface</hardwareInterface>
+    <mechanicalReduction>1</mechanicalReduction>
+  </actuator>
 </transmission>
 <transmission name="tran5">
-<type>transmission_interface/SimpleTransmission</type>
-<joint name="hand_to_left_finger">
-  <hardwareInterface>EffortJointInterface</hardwareInterface>
-</joint>
-<actuator name="motor5">
-  <hardwareInterface>EffortJointInterface</hardwareInterface>
-  <mechanicalReduction>1</mechanicalReduction>
-</actuator>
+  <type>transmission_interface/SimpleTransmission</type>
+  <joint name="hand_to_left_finger">
+    <hardwareInterface>EffortJointInterface</hardwareInterface>
+  </joint>
+  <actuator name="motor5">
+    <hardwareInterface>EffortJointInterface</hardwareInterface>
+    <mechanicalReduction>1</mechanicalReduction>
+  </actuator>
 </transmission>
 </robot>
